File: schematics/c3lingo-interpreter-unit.sch (KiCad schematic (older format))
At the start: 68 parts, among them J1 Headphone 1, J2 Mic 1, J3 Mix Line-Out, J4 Stage Line-In, J5 Mains_PowerTwist, SW1 Mute_1, SW2 OnAir_1, U1 LM833N, U2 NE5534, U3 LM833N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

Commit message: Schematic: Bugfixes, VU meter draft, first development PCB draft
Parts:
- removed C21: 10-100 uF, symbol Device:C
- removed C22: 250pF, symbol Device:CP
- removed C23: 0.05uF, symbol Device:C
- removed C24: 10uF, symbol Device:CP
- removed PS1: TXL 035-1515D, symbol Converter_ACDC:TMLM04253
- removed R24: 10K, Potentiometer_THT:Potentiometer_Vishay_148-149_Single_Horizontal, symbol Device:R_POT
- removed R25: 10K, symbol Device:R
- removed U7: LM386N-4, symbol Amplifier_Audio:LM386
- added C21: 10uF, Capacitor_THT:CP_Radial_D10.0mm_P5.00mm, symbol Device:CP
- added JP1: Stage Hot, Connector_PinHeader_2.54mm:PinHeader_1x03_P2.54mm_Vertical, symbol Jumper:Jumper_3_Bridged12
- added JP2: Stage Cold, Connector_PinHeader_2.54mm:PinHeader_1x03_P2.54mm_Vertical, symbol Jumper:Jumper_3_Bridged12
- added JP3: Stage Out, Connector_PinHeader_2.54mm:PinHeader_1x03_P2.54mm_Vertical, symbol Jumper:Jumper_3_Bridged12
- C1, C6, C9: footprint (none) -> Capacitor_THT:CP_Radial_D10.0mm_P5.00mm
- C10, C11, C12, C13, C14, C15, C16, C17, C18, C19, C2, C20, C25, C3, C4, C5, C8: footprint (none) -> Capacitor_THT:C_Disc_D5.0mm_W2.5mm_P5.00mm
- C7: value 4.7pF -> 10nF; footprint (none) -> Capacitor_THT:C_Disc_D5.0mm_W2.5mm_P5.00mm
- J1, J2, J3, J4, SW2: footprint (none) -> Connector_PinHeader_2.54mm:PinHeader_1x04_P2.54mm_Vertical
- J5: value Mains_PowerTwist -> PowerSupply; footprint (none) -> TerminalBlock_MetzConnect:TerminalBlock_MetzConnect_Type073_RT02603HBLU_1x03_P5.08mm_Horizontal
- R1, R10, R12, R13, R14, R15, R16, R17, R18, R19, R20, R21, R22, R23, R26, R6, R7, R8, R9: footprint (none) -> Resistor_THT:R_Axial_DIN0207_L6.3mm_D2.5mm_P10.16mm_Horizontal
- R11, R2: value 324K 1% -> 330K 1%; footprint (none) -> Resistor_THT:R_Axial_DIN0207_L6.3mm_D2.5mm_P10.16mm_Horizontal
- R5: value 27.5K 1% -> 27K 1%; footprint (none) -> Resistor_THT:R_Axial_DIN0207_L6.3mm_D2.5mm_P10.16mm_Horizontal
- SW1: footprint (none) -> Connector_PinHeader_2.54mm:PinHeader_1x02_P2.54mm_Vertical; symbol Switch:SW_Push_Open -> Switch:SW_Push
- U1, U2, U3, U4, U5, U6: footprint Package_DIP:DIP-8_W7.62mm -> Package_DIP:DIP-8_W7.62mm_Socket_LongPads
Connections:
- net Earth_Protective is gone; now on net -15V: J5.3 (Pin_3)
- net +15V: now also C8.1, C9.1, J5.1 (Pin_1); no longer C1.1, C2.2
- net -15V: now also C1.2, C2.2; no longer C8.2, C9.2
- net GNDREF: now also C1.1, C8.2, C9.2, J5.2 (Pin_2), R4.1; no longer C1.2, C8.1, C9.1
- net Mic1: now also SW1.2
- net at R10.1, R11.2, R5.2: now also U2.3 (+); no longer U2.2 (-)
- net at R1.1, R2.2, R5.1: now also U2.2 (-); no longer U2.3 (+)
- net at R17.1, U4.1: now also JP3.1 (A); no longer R20.2
- net at J4.3, J4.R: now also JP2.2 (C); no longer R21.2
- net at J4.2, J4.T: now also JP1.2 (C); no longer R18.2
- net at C25.2, R26.2, U1.2 (-): now also SW1.1, C21.2; no longer R6.1
- net at C3.2, R4.2, R9.1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: now also R3.1; no longer R3.3
- net at U6.2 (IN-): now also JP1.3 (B)
- net at U6.3 (IN+): now also JP2.3 (B)
- net at U6.5 (SENSE), U6.6 (OUTPUT): now also JP3.3 (B)
- new net: C21.1, R6.1
- new net: JP1.1 (A), R18.2
- new net: JP2.1 (A), R21.2
- new net: JP3.2 (C), R20.2
- no-connect marks 12 -> 13
Other:
- note added: "Headphone gain either at mix (summing)\nor at the driver"
- note added: "TODO Headphone driver\nGain: TODO"
- note added: "TODO: On-Air buttons"
- note added: "TODO: Rotation direction of potentiometers!\n(counter-clockwise less gain, clockwise more gain)"
- note removed: "Headphone driver\nGain: TODO"
- note removed: "TODO: On-Air and Mute buttons"
- note removed: "TODO: VU Meter !!!!"
- moved on the sheet: C14, C15, C16, C19, C20, C25, J4A, J4B, J5, R17, R18, R19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
