File: schematics/c3lingo_unit-assembly/c3lingo_unit-channel/c3lingo_unit-channel.sch (KiCad schematic (older format))
At the start: 92 parts, among them J1 Headphone 1, J2 Mic 1, J3 Mix Line-Out, J4 Stage Line-In, J5 PowerSupply, J6 PowerSupply, SW1 Mute_1, SW2 OnAir_1, U1 LM833N, U2 NE5534, U3 LM833N, U4 LM833N, U5 DRV134PA, U7 LM386N-4

Commit message: [TIDY] Split old design in new hierarchal layout
TODO: Shrink channel strip to A4 paper size, integrate VU meter
Parts:
- removed C10: 22pF, Capacitor_THT:C_Disc_D5.0mm_W2.5mm_P5.00mm, symbol Device:C
- removed C11, C12, C15, C16: 100nF, Capacitor_THT:C_Disc_D5.0mm_W2.5mm_P5.00mm, symbol Device:C
- removed C14: 47pF, Capacitor_THT:C_Disc_D5.0mm_W2.5mm_P5.00mm, symbol Device:C
- removed C17, C18: 1uF, Capacitor_THT:C_Disc_D5.0mm_W2.5mm_P5.00mm, symbol Device:C
- removed C27: 220pF, Capacitor_THT:C_Disc_D5.0mm_W2.5mm_P5.00mm, symbol Device:C
- removed J3: Mix Line-Out, Connector_PinHeader_2.54mm:PinHeader_1x04_P2.54mm_Vertical, symbol Connector:XLR3_Ground
- removed J4: Stage Line-In, Connector_PinHeader_2.54mm:PinHeader_1x04_P2.54mm_Vertical, symbol Connector:XLR3_AudioJack3_Combo_Ground
- removed J6: PowerSupply, TerminalBlock_MetzConnect:TerminalBlock_MetzConnect_Type073_RT02603HBLU_1x03_P5.08mm_Horizontal, symbol Connector:Conn_01x03_Male
- removed R12, R13, R14, R16, R19: 22K, Resistor_THT:R_Axial_DIN0207_L6.3mm_D2.5mm_P10.16mm_Horizontal, symbol Device:R
- removed R17, R18, R21, R23, R3, R8: 10K, Resistor_THT:R_Axial_DIN0207_L6.3mm_D2.5mm_P10.16mm_Horizontal, symbol Device:R
- removed R20: 47K, Resistor_THT:R_Axial_DIN0207_L6.3mm_D2.5mm_P10.16mm_Horizontal, symbol Device:R
- removed R4: 3.3K, Resistor_THT:R_Axial_DIN0207_L6.3mm_D2.5mm_P10.16mm_Horizontal, symbol Device:R
- removed RV1: 100K, Potentiometer_THT:Potentiometer_Vishay_T73XX_Horizontal, symbol Device:R_POT
- removed TP10: Mic2, TestPoint:TestPoint_THTPad_D2.0mm_Drill1.0mm, symbol Connector:TestPoint
- removed TP11: Mic3, TestPoint:TestPoint_THTPad_D2.0mm_Drill1.0mm, symbol Connector:TestPoint
- removed TP6: MicSum, TestPoint:TestPoint_THTPad_D2.0mm_Drill1.0mm, symbol Connector:TestPoint
- removed TP8: Stage, TestPoint:TestPoint_THTPad_D2.0mm_Drill1.0mm, symbol Connector:TestPoint
- removed TP9: Mic1, TestPoint:TestPoint_THTPad_D2.0mm_Drill1.0mm, symbol Connector:TestPoint
- removed U3, U4: LM833N, Package_DIP:DIP-8_W7.62mm_Socket_LongPads, symbol Amplifier_Operational:LM358
- removed U5: DRV134PA, Package_DIP:DIP-8_W7.62mm_Socket_LongPads, symbol JBeyerstedt-Library:DRV134PA
- J1: value Headphone 1 -> Headphone X
- J2: value Mic 1 -> Mic X In
Connections:
- net labels added: Monitor_OthersA, Monitor_OthersB, Monitor_Own, Monitor_Stage, PreampOut
- net labels removed: Mic1, Stage
- wire segments 342 -> 207
- no-connect marks 7 -> 10
Other:
- note added: "HP Filter 350 Hz\nf_c = 1/(2*PI*R*C)\nTODO: lower freq!!!"
- note removed: "Balanced Line Input Converter\nGain: 1\n220pF for HF rolloff (20 kHz)"
- note removed: "HP Filter 350 Hz\nf_c = 1/(2*PI*R*C)"
- note removed: "Input Module\nGain: -6 to +8 dB\nGain = (R_pot + R_22k) / R_47k\nLP_filter(R_pot): 130 - 22 kHz"
- note removed: "Line driver\nGain: 6 dB"
- note removed: "Mic2"
- note removed: "Mic3"
- note removed: "Summing Module\nGain: 0 dB"

Commit message: [TIDY] Channel Strip: Integrate VU Meter
Parts:
- removed TP1: Mic1, TestPoint:TestPoint_THTPad_D2.0mm_Drill1.0mm, symbol Connector:TestPoint
- added C64: 1uF, Capacitor_THT:CP_Radial_D5.0mm_P2.50mm, symbol Device:CP
- added C65: 47uF, Capacitor_THT:CP_Radial_D10.0mm_P2.50mm_P5.00mm, symbol Device:CP
- added C66, C67, C68, C69, C70: 100nF, Capacitor_THT:C_Disc_D5.0mm_W2.5mm_P5.00mm, symbol Device:C
- added D13: -32 rd, LED_THT:LED_D5.0mm, symbol Device:LED
- added D14: -28 rd, LED_THT:LED_D5.0mm, symbol Device:LED
- added D15: -24 rd, LED_THT:LED_D5.0mm, symbol Device:LED
- added D16: -20 rd, LED_THT:LED_D5.0mm, symbol Device:LED
- added D17: -16 ye, LED_THT:LED_D5.0mm, symbol Device:LED
- added D18: -12 ye, LED_THT:LED_D5.0mm, symbol Device:LED
- added D19: -8 gn, LED_THT:LED_D5.0mm, symbol Device:LED
- added D20: -4 gn, LED_THT:LED_D5.0mm, symbol Device:LED
- added D21: 0 gn, LED_THT:LED_D5.0mm, symbol Device:LED
- added D22: +4 ye, LED_THT:LED_D5.0mm, symbol Device:LED
- added D23: +8 ye, LED_THT:LED_D5.0mm, symbol Device:LED
- added D24: +12 rd, LED_THT:LED_D5.0mm, symbol Device:LED
- added D25, D26: 1N4148, Diode_THT:D_DO-35_SOD27_P10.16mm_Horizontal, symbol Device:D
- added J13: Inputs, Connector_PinHeader_2.54mm:PinHeader_1x04_P2.54mm_Vertical, symbol Connector:Conn_01x04_Male
- added J14: Output, Connector_PinHeader_2.54mm:PinHeader_1x02_P2.54mm_Vertical, symbol Connector:Conn_01x02_Male
- added JP1, JP2: GND_JMP, Jumper:SolderJumper-2_P1.3mm_Open_TrianglePad1.0x1.5mm, symbol Jumper:SolderJumper_2_Open
- added R68, R93: 3.9K, Resistor_THT:R_Axial_DIN0207_L6.3mm_D2.5mm_P10.16mm_Horizontal, symbol Device:R
- added R69, R70, R71, R72, R73, R74, R75, R76, R77, R78, R79, R80, R88: 390R, Resistor_THT:R_Axial_DIN0207_L6.3mm_D2.5mm_P10.16mm_Horizontal, symbol Device:R
- added R81, R90: 1K, Resistor_THT:R_Axial_DIN0207_L6.3mm_D2.5mm_P10.16mm_Horizontal, symbol Device:R
- added R82, R84: 68R, Resistor_THT:R_Axial_DIN0207_L6.3mm_D2.5mm_P10.16mm_Horizontal, symbol Device:R
- added R83: 39R, Resistor_THT:R_Axial_DIN0207_L6.3mm_D2.5mm_P10.16mm_Horizontal, symbol Device:R
- added R85: 100R, Resistor_THT:R_Axial_DIN0207_L6.3mm_D2.5mm_P10.16mm_Horizontal, symbol Device:R
- added R86: 150R, Resistor_THT:R_Axial_DIN0207_L6.3mm_D2.5mm_P10.16mm_Horizontal, symbol Device:R
- added R87: 270R, Resistor_THT:R_Axial_DIN0207_L6.3mm_D2.5mm_P10.16mm_Horizontal, symbol Device:R
- added R89: 680R, Resistor_THT:R_Axial_DIN0207_L6.3mm_D2.5mm_P10.16mm_Horizontal, symbol Device:R
- added R91: 1.5K, Resistor_THT:R_Axial_DIN0207_L6.3mm_D2.5mm_P10.16mm_Horizontal, symbol Device:R
- added R92, R94: 2.7K, Resistor_THT:R_Axial_DIN0207_L6.3mm_D2.5mm_P10.16mm_Horizontal, symbol Device:R
- added R95: 100K, Resistor_THT:R_Axial_DIN0207_L6.3mm_D2.5mm_P10.16mm_Horizontal, symbol Device:R
- added RV16: 50K, Potentiometer_THT:Potentiometer_Vishay_T73XX_Horizontal, symbol Device:R_POT
- added SW?: OnAir_1, symbol Switch:SW_DPDT_x2
- added U13, U14, U15: LM339, Package_DIP:DIP-14_W7.62mm_Socket_LongPads, symbol Comparator:LM339
- added U16: LM833N, Package_DIP:DIP-8_W7.62mm_Socket_LongPads, symbol Amplifier_Operational:LM358
- J5: footprint TerminalBlock_MetzConnect:TerminalBlock_MetzConnect_Type073_RT02603HBLU_1x03_P5.08mm_Horizontal -> TerminalBlock_MetzConnect:TerminalBlock_MetzConnect_Type101_RT01604HBWC_1x04_P5.08mm_Horizontal; symbol Connector:Conn_01x03_Male -> Connector:Conn_01x04_Male
- SW1: footprint Connector_PinHeader_2.54mm:PinHeader_1x02_P2.54mm_Vertical -> (none); Model NKK Switches UB15{NBK,NK}{W,G}{01,03}N-C -> APEM 1415NC6
- SW2: footprint Connector_PinHeader_2.54mm:PinHeader_1x04_P2.54mm_Vertical -> (none); symbol Switch:SW_SPST_LED -> Switch:SW_DPDT_x2; Model E-Switch LP11EE1NCSYG -> APEM MHPS2273
- TP3: value Mic1 -> MicX
- TP4: value Mic2 -> MicA
- TP5: value Mic3 -> MicB
Connections:
- net PreampOut is gone; now on net VUMeter: C25.1, RV11.2, SW1.2, U1.1
- net +15V: now also J5.2 (Pin_2), C67.2, C68.1, C69.1, C70.1, D13.2 (A), D14.2 (A), D15.2 (A), D16.2 (A), D17.2 (A), D18.2 (A), D19.2 (A), D20.2 (A), D21.2 (A), D22.2 (A), D23.2 (A), D24.2 (A), R94.2, U13.3 (V+), U14.3 (V+), U15.3 (V+), U16.8 (V+); no longer C19.1, J5.1 (Pin_1), R15.2, R22.1
- net -15V: now also C66.2, U16.4 (V-)
- net GND: now also J5.1 (Pin_1), C65.2, C66.1, C67.1, C68.2, C69.2, C70.2, J13.1 (Pin_1), J14.1 (Pin_1), JP1.1 (A), JP2.1 (A), R82.1, R95.2, RV16.3, U13.12 (V-), U14.12 (V-), U15.12 (V-), U16.3 (+); no longer J1.G, J2.G, J5.2 (Pin_2)
- net Monitor_OthersA: now also J13.3 (Pin_3)
- net Monitor_OthersB: now also J13.4 (Pin_4)
- net Monitor_Stage: now also J13.2 (Pin_2)
- net Monitor_Own renamed VUMeter
- net VUMeter: now also J14.2 (Pin_2), RV16.1
- new net: R80.2, U15.2
- new net: C65.1, D26.1 (K), R68.1, R95.1, U13.10 (-), U13.4 (-), U13.6 (-), U13.8 (-), U14.10 (-), U14.4 (-), U14.6 (-), U14.8 (-), U15.10 (-), U15.4 (-), U15.6 (-), U15.8 (-)
- new net: R93.2, R94.1, U15.5 (+)
- new net: R79.2, U15.1
- new net: R92.2, R93.1, U15.7 (+)
- new net: R91.2, R92.1, U15.11 (+)
- new net: R78.2, U15.13
- new net: R77.2, U15.14
- new net: R90.2, R91.1, U15.9 (+)
- new net: R89.2, R90.1, U14.5 (+)
- new net: R76.2, U14.2
- new net: R75.2, U14.1
- new net: R88.2, R89.1, U14.7 (+)
- new net: R87.2, R88.1, U14.11 (+)
- new net: R74.2, U14.13
- new net: R73.2, U14.14
- new net: R86.2, R87.1, U14.9 (+)
- new net: R85.2, R86.1, U13.5 (+)
- new net: R72.2, U13.2
- new net: R71.2, U13.1
- new net: R84.2, R85.1, U13.7 (+)
- new net: R83.2, R84.1, U13.11 (+)
- new net: R70.2, U13.13
- new net: R69.2, U13.14
- new net: R82.2, R83.1, U13.9 (+)
- new net: D24.1 (K), R80.1
- new net: D23.1 (K), R79.1
- new net: D22.1 (K), R78.1
- new net: D21.1 (K), R77.1
- new net: D20.1 (K), R76.1
- new net: D19.1 (K), R75.1
- new net: D18.1 (K), R74.1
- new net: D17.1 (K), R73.1
- new net: D16.1 (K), R72.1
- new net: D15.1 (K), R71.1
- new net: D14.1 (K), R70.1
- new net: D13.1 (K), R69.1
- new net: D25.2 (A), R68.2, R81.2, U16.2 (-)
- new net: D25.1 (K), D26.2 (A), U16.1
- new net: C64.1, RV16.2
- new net: C64.2, R81.1
- new net GNDREF: J1.G, J2.G, JP1.2 (B), JP2.2 (B)
- new net Pxx_V: C19.1, J5.4 (Pin_4), R15.2, R22.1
- no-connect marks 10 -> 6
Other:
- note added: "+0 dBu"
- note added: "+12 dBu"
- note added: "+4 dBu"
- note added: "+8 dBu"
- note added: "-12 dBu"
- note added: "-16 dBu"
- note added: "-20 dBu"
- note added: "-24 dBu"
- note added: "-28 dBu"
- note added: "-32 dBu"
- note added: "-4 dBu"
- note added: "-8 dBu"
- note added: "48V: R = 6.81K\n24V: R = 1.2K\n12V: R = 680R"
- note added: "Buffer/ Rectifier\nGain: 3.9"
- note added: "For Input Gain of 3.9:\n2700 Ω: 11,99 dBu\n3900 Ω: 8,12 dBu\n2700 Ω: 3,86 dBu\n1500 Ω: 0,1 dBu\n1000 Ω: -3,8 dBu\n680 Ω: -8,03 dBu\n390 Ω: -11,89 dBu\n270 Ω: -16,17 dBu\n150 Ω: -19,95 dBu\n100 Ω: -23,87 dBu\n68 Ω: -28,15 dBu\n39 Ω: -32,08 dBu\n68 Ω to ground\n\n1.11 mA @ 15V\n(13.565 kΩ)"
- note added: "Signal Smoothing\nTODO: Remove all together!?"
- note added: "TODO: Better use 5V?\nrd: 2.3 V (390R @15V)\ngn: 2.4 V (390R @15V)\nye: 2.6 V (390R @15V)"

Commit message: Schematics: Add missing functionality, add footprints, fix todos
- Add On-Air button
- Lower frequency for the input HPF
- (final) button footprints
- (final) potentiometer values and footprints
Parts:
- removed JP1: GND_JMP, Jumper:SolderJumper-2_P1.3mm_Open_TrianglePad1.0x1.5mm, symbol Jumper:SolderJumper_2_Open
- added D301: On-Air (rd), LED_THT:LED_D5.0mm, symbol Device:LED
- added H301, H302, H303, H305, H306: MountingHole, MountingHole:MountingHole_3.2mm_M3, symbol Mechanical:MountingHole
- added J306: PowerSupply, TerminalBlock_Phoenix:TerminalBlock_Phoenix_PTSM-0,5-4-2.5-H-THR_1x04_P2.50mm_Horizontal, symbol Connector:Conn_01x04_Male
- added J307: Interconnect, TerminalBlock_Phoenix:TerminalBlock_Phoenix_PTSM-0,5-3-2.5-H-THR_1x03_P2.50mm_Horizontal, symbol Connector:Conn_01x03_Female
- added J308: Interconnect, TerminalBlock_Phoenix:TerminalBlock_Phoenix_PTSM-0,5-3-2.5-H-THR_1x03_P2.50mm_Horizontal, symbol Connector:Conn_01x03_Male
- added R306: 390R, Resistor_THT:R_Axial_DIN0207_L6.3mm_D2.5mm_P10.16mm_Horizontal, symbol Device:R
- C301: renamed from C1; footprint Capacitor_THT:CP_Radial_D10.0mm_P5.00mm -> Capacitor_THT:CP_Radial_D6.3mm_P2.50mm
- C302: renamed from C21; footprint Capacitor_THT:CP_Radial_D10.0mm_P5.00mm -> Capacitor_THT:CP_Radial_D6.3mm_P2.50mm
- C307: renamed from C13; value 1uF -> 1uF/ 63V
- C308: renamed from C23; footprint Capacitor_THT:CP_Radial_D10.0mm_P5.00mm -> Capacitor_THT:CP_Radial_D6.3mm_P2.50mm
- C310: renamed from C24; value 220uF -> 220uF lowESR
- C311: renamed from C19; value 100uF -> 100uF/ 63V
- C313: renamed from C20; value 1uF -> 1uF/ 63V
- C318: renamed from C9; footprint Capacitor_THT:CP_Radial_D10.0mm_P5.00mm -> Capacitor_THT:CP_Radial_D6.3mm_P2.50mm
- C319: renamed from C64; footprint Capacitor_THT:CP_Radial_D5.0mm_P2.50mm -> Capacitor_THT:CP_Radial_D5.0mm_P2.00mm
- C320: renamed from C65; footprint Capacitor_THT:CP_Radial_D10.0mm_P2.50mm_P5.00mm -> Capacitor_THT:CP_Radial_D6.3mm_P2.50mm
- D306: renamed from D13; value -32 rd -> rd
- D307: renamed from D14; value -28 rd -> rd
- D308: renamed from D15; value -24 rd -> rd
- D309: renamed from D16; value -20 rd -> rd
- D310: renamed from D17; value -16 ye -> ye
- D311: renamed from D18; value -12 ye -> ye
- D312: renamed from D19; value -8 gn -> gn
- D313: renamed from D20; value -4 gn -> gn
- D314: renamed from D21; value 0 gn -> gn
- D315: renamed from D22; value +4 ye -> ye
- D316: renamed from D23; value +8 ye -> ye
- D317: renamed from D24; value +12 rd -> rd
- J301: renamed from J2; footprint Connector_PinHeader_2.54mm:PinHeader_1x04_P2.54mm_Vertical -> Connector_Audio:Jack_XLR_Neutrik_NC3FAAH2_Horizontal; Model XLR (female) -> NC3FAAH2 (Horiz. Male)
- J302: renamed from J1; footprint Connector_PinHeader_2.54mm:PinHeader_1x04_P2.54mm_Vertical -> Connector_Audio:Jack_6.35mm_Neutrik_NMJ6HFD2_Horizontal; Model 6.3 mm Jack (female) -> NYS216G (Horiz.)
- J303: renamed from J5; footprint TerminalBlock_MetzConnect:TerminalBlock_MetzConnect_Type101_RT01604HBWC_1x04_P5.08mm_Horizontal -> TerminalBlock_Phoenix:TerminalBlock_Phoenix_PTSM-0,5-4-2.5-H-THR_1x04_P2.50mm_Horizontal; Model (none) -> PTSM 0,5/ 4-2,5-H THR
- J304: renamed from J13; footprint Connector_PinHeader_2.54mm:PinHeader_1x04_P2.54mm_Vertical -> TerminalBlock_Phoenix:TerminalBlock_Phoenix_PTSM-0,5-4-2.5-H-THR_1x04_P2.50mm_Horizontal; Model TODO: Actual Connector -> PTSM 0,5/ 4-2,5-H THR
- J305: renamed from J14; footprint Connector_PinHeader_2.54mm:PinHeader_1x02_P2.54mm_Vertical -> TerminalBlock_Phoenix:TerminalBlock_Phoenix_PTSM-0,5-2-2.5-H-THR_1x02_P2.50mm_Horizontal; Model TODO: Actual Connector -> PTSM 0,5/ 2-2,5-H THR
- R305: renamed from R26; value 270R -> 56R
- R310: renamed from R6; value 1.5K -> 330R
- R312: renamed from R7; value 470R -> 820R
- RV301: renamed from RV13; footprint JBeyerstedt-Library:Potentiometer_Alps_RK11K_Single_Horizontal -> c3lingo_unit-footprints:Potentiometer_Alps_RK09K_Double_Vertical; Model Alps RK11K1120-A503 -> Alps RK09K12C0A2S (dual, vert.)
- RV302: renamed from RV11; value 50K log. -> 10K log.; footprint JBeyerstedt-Library:Potentiometer_Alps_RK11K_Single_Horizontal -> Potentiometer_THT:Potentiometer_Alps_RK09K_Single_Vertical; Model Alps RK11K1120-A503 -> Alps RK09K1130AJ3 (single, vert.)
- RV303: renamed from RV14; footprint JBeyerstedt-Library:Potentiometer_Alps_RK11K_Single_Horizontal -> c3lingo_unit-footprints:Potentiometer_Alps_RK09K_Double_Vertical; Model Alps RK11K1120-A503 -> Alps RK09K12C0A2S (dual, vert.)
- RV304: renamed from RV19; footprint JBeyerstedt-Library:Potentiometer_Alps_RK11K_Single_Horizontal -> Potentiometer_THT:Potentiometer_Alps_RK09K_Single_Horizontal; Model Alps RK11K1120-A503 -> RK09K1110B1R (single, horiz.)
- RV305: renamed from RV15; footprint Potentiometer_THT:Potentiometer_Alps_RK09L_Double_Horizontal -> c3lingo_unit-footprints:Potentiometer_Alps_RK09K_Double_Vertical; Model Alps RK14K12B0A0R / RK09L1220 -> Alps RK09K12C0A2S (dual, vert.)
- RV306: renamed from RV16; Model Vishay M64{Y,Z}503K -> Vishay M64Y503
- SW301: renamed from SW2; value OnAir_1 -> OnAir_X; footprint (none) -> c3lingo_unit-footprints:SW_APEM_MHPS2273_DPDT
- SW301: renamed from SW?; value OnAir_1 -> OnAir_X; footprint (none) -> c3lingo_unit-footprints:SW_APEM_MHPS2273_DPDT; Model APEM MHPS2273 -> APEM MHPS2273 (US)/ PHAP4673 (EU)
- SW302: renamed from SW1; value Mute_1 -> Mute_X; footprint (none) -> Connector_PinHeader_2.54mm:PinHeader_1x02_P2.54mm_Vertical; Model APEM 1415NC6 -> APEM 1415NC6 (solder lug)
- renumbered C3 to C303, C2 to C304, C22 to C305, C25 to C306, C6 to C309, C26 to C312, C7 to C314, C8 to C315, C4 to C316, C5 to C317, C66 to C321, C67 to C322, C68 to C323, C69 to C324, C70 to C325, D2 to D302, D1 to D303, D3 to D304, D4 to D305, D25 to D318, D26 to D319, JP2 to JP302, R86 to R138, R28 to R301, R9 to R302, R1 to R303, R2 to R304, R15 to R307, R29 to R308, R5 to R309, R22 to R311, R24 to R313, R10 to R314, R11 to R315, R25 to R316, R30 to R317, R27 to R318, R31 to R319, R68 to R320, R69 to R321, R70 to R322, R71 to R323, R72 to R324, R73 to R325, R74 to R326, R75 to R327, R76 to R328, R77 to R329, R78 to R330, R79 to R331, R80 to R332, R81 to R333, R82 to R334, R83 to R335, R84 to R336, R85 to R337, R87 to R339, R88 to R340, R89 to R341, R90 to R342, R91 to R343, R92 to R344, R93 to R345, R94 to R346, R95 to R347, TP2 to TP301, TP3 to TP302, TP4 to TP303, TP5 to TP304, U2 to U301, U1 to U302, U7 to U303, U16 to U304, U13 to U305, U14 to U306, U15 to U307
Connections:
- net VUMeter is gone; now on net PreampOut: C306.1, J305.2 (Pin_2), RV302.2, RV303.3, RV306.1, SW302.2, TP302.1, U302.1
- net +15V: now also C305.1, J306.2 (Pin_2); no longer C305.2, D306.2 (A), D307.2 (A), D308.2 (A), D309.2 (A), D310.2 (A), D311.2 (A), D312.2 (A), D313.2 (A), D314.2 (A), D315.2 (A), D316.2 (A), D317.2 (A)
- net -15V: now also J306.3 (Pin_3)
- net GND: now also C305.2, R312.2, U304.5 (+), J306.1 (Pin_1), J307.1 (Pin_1), J308.1 (Pin_1), R306.2; no longer C305.1, R312.1, U304.3 (+)
- net GNDREF: no longer J302.G
- net at R303.1, R309.1, U301.2 (-): now also R304.1; no longer R304.2
- net at C309.1, U301.6: now also R304.2; no longer R304.1
- net at C307.1, J301.2: now also R307.2; no longer R307.1
- net at C313.1, J301.3: now also R311.1; no longer R311.2
- net at C306.2, R305.2, R310.1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: now also SW301.2 (B)
- net SumOut: now reaches C303.1, R302.1, U302.7
- net SumOut: now also J308.2 (Pin_2); no longer R313.1
- net at D318.2 (A), R320.2, R333.2: now also U304.6 (-); no longer U304.2 (-)
- net at D318.1 (K), D319.2 (A): now also U304.7; no longer U304.1
- net PreampOut: now reaches SW301.1 (A)
- net V_LED: now reaches SW301.5 (B)
- net V_LED: now also D306.2 (A), D307.2 (A), D308.2 (A), D309.2 (A), D310.2 (A), D311.2 (A), D312.2 (A), D313.2 (A), D314.2 (A), D315.2 (A), D316.2 (A), D317.2 (A), J303.4 (Pin_4)
- net at SW301.6 (C): now also D301.2 (A)
- removed net Pxx_V: C311.1, J303.4 (Pin_4), R307.2, R311.1
- new net: D301.1 (K), R306.1
- new net AmpIn: J307.2 (Pin_2), R313.1
- new net MicGainIn: J308.3 (Pin_3), R310.2
- new net MicPreOut: C309.2, J307.3 (Pin_3), R312.1
- new net V_Phant: C311.1, J306.4 (Pin_4), R307.1, R311.2
- no-connect marks 6 -> 9
Other:
- note added: "For Input Gain of 3.9\nand VCC = 15V:\n2700 Ω: 11,99 dBu\n3900 Ω: 8,12 dBu\n2700 Ω: 3,86 dBu\n1500 Ω: 0,1 dBu\n1000 Ω: -3,8 dBu\n680 Ω: -8,03 dBu\n390 Ω: -11,89 dBu\n270 Ω: -16,17 dBu\n150 Ω: -19,95 dBu\n100 Ω: -23,87 dBu\n68 Ω: -28,15 dBu\n39 Ω: -32,08 dBu\n68 Ω to ground\n\n1.11 mA @ 15V\n(13.565 kΩ)"
- note added: "Gain Range (Rin @input, R1 + Rpot @feedback):\nGain_min = R1 / Rin (Rpot_min = 0)\nGain_max = (R1+Rpot_max) / Rin\n=> R1 = -(Rpot * Gain_min) / (Gain_min - Gain_max)\n=> R2 = -(Rpot) / (Gain_min - Gain_max)"
- note added: "HP Filter 200 Hz\nf_c = 1/(2*PI*R*C)\n160 Hz @ 1K"
- note added: "Mute/ On-Air:\nClosed = -inf Gain\nMute: NO (un-muted)\nOn-Air: NC (mic muted) / push to activate"
- note added: "TODO: Change to 10 uF?"
- note added: "TODO: Try with V_LED = 5V\nrd: 2.3 V (390R @15V)\ngn: 2.4 V (390R @15V)\nye: 2.6 V (390R @15V)"
- note removed: "For Input Gain of 3.9:\n2700 Ω: 11,99 dBu\n3900 Ω: 8,12 dBu\n2700 Ω: 3,86 dBu\n1500 Ω: 0,1 dBu\n1000 Ω: -3,8 dBu\n680 Ω: -8,03 dBu\n390 Ω: -11,89 dBu\n270 Ω: -16,17 dBu\n150 Ω: -19,95 dBu\n100 Ω: -23,87 dBu\n68 Ω: -28,15 dBu\n39 Ω: -32,08 dBu\n68 Ω to ground\n\n1.11 mA @ 15V\n(13.565 kΩ)"
- note removed: "HP Filter 350 Hz\nf_c = 1/(2*PI*R*C)\nTODO: lower freq!!!"
- note removed: "TODO: Better use 5V?\nrd: 2.3 V (390R @15V)\ngn: 2.4 V (390R @15V)\nye: 2.6 V (390R @15V)"
- note removed: "TODO: C at pin 7 has\nno audible effect"
- note removed: "TODO: On-Air button LEDs\n(actually one rd, one gn,\nwith common anode)"
- moved on the sheet: C301, C302, C303, C304, C305, C306, C307, C308, C309, C310, C311, C312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
