File: schematics/c3lingo_unit-assembly/c3lingo_unit-channel/c3lingo_unit-channel.kicad_sch (KiCad schematic)
At the start: 124 parts, among them J301 Mic X In, J302 Headphone X, J303 Interconnect, J304 Interconnect, J305 PowerSupply, J306 PowerSupply, J307 Inputs, J308 Output, SW301 OnAir_X, SW302 Mute_X, U301 NE5534, U302 LM833N, U303 LM386N-4, U304 LM339, U305 LM339, U306 LM339, U307 LM833N

Commit message: Schematics: Fix multiple issues with initial prototype
- Removed high-pass filter between microphone pre-amp and gain as it made things sound worse
- Removed low-pass filter before VU meter as it looked fine without
- Connect VU meter to +15 V directly as 5 V didn't work
- Footprint of the gain potentiometer (Alps RK09) seems to be fixed with the KiCad 6 library
Parts:
- removed C309: 1uF, Capacitor_THT:CP_Radial_D5.0mm_P2.00mm, symbol Device:C_Polarized
- removed C320: 47uF, Capacitor_THT:CP_Radial_D6.3mm_P2.50mm, symbol Device:C_Polarized
- removed R312: 820R, Resistor_THT:R_Axial_DIN0207_L6.3mm_D2.5mm_P10.16mm_Horizontal, symbol Device:R
- removed R347: 100K, Resistor_THT:R_Axial_DIN0207_L6.3mm_D2.5mm_P10.16mm_Horizontal, symbol Device:R
- C306: value 100nF -> 10nF
- J306: footprint TerminalBlock_Phoenix:TerminalBlock_Phoenix_PTSM-0,5-4-2.5-H-THR_1x04_P2.50mm_Horizontal -> TerminalBlock_Phoenix:TerminalBlock_Phoenix_PTSM-0,5-4-2.5-H-THR_1x03_P2.50mm_Horizontal; symbol Connector:Conn_01x04_Male -> Connector:Conn_01x03_Male; Model PTSM 0,5/ 4-2,5-H THR -> PTSM 0,5/ 3-2,5-H THR
- J308: symbol Connector:Conn_01x02_Male -> Connector:Conn_01x04_Male; Model PTSM 0,5/ 2-2,5-H THR -> PTSM 0,5/ 4-2,5-H THR
- R306: value 390R -> 680R
Connections:
- net +15V: now also D306.2 (A), D307.2 (A), D308.2 (A), D309.2 (A), D310.2 (A), D311.2 (A), D312.2 (A), D313.2 (A), D314.2 (A), D315.2 (A), D316.2 (A), D317.2 (A), SW301.5 (B)
- net MicPreOut: now also R304.2, U301.6
- net PreampOut: now also J308.3 (Pin_3), J308.4 (Pin_4)
- removed net V_LED: D306.2 (A), D307.2 (A), D308.2 (A), D309.2 (A), D310.2 (A), D311.2 (A), D312.2 (A), D313.2 (A), D314.2 (A), D315.2 (A), D316.2 (A), D317.2 (A), J306.4 (Pin_4), SW301.5 (B)
Other:
- note removed: "Bridge V_LED to +15V (5V V_LED didn’t work)"
- note removed: "DNP R312 and replace C309 with a jumper!"
- note removed: "HP Filter 200 Hz f_c = 1/(2*PI*R*C) 160 Hz @ 1K"
- note removed: "PCB Errata: - R302 (R102 on PCB) has pins 1 and 3 swapped. Connect R305 (R105) directly to the left potentiometer pin! - The ground plane at the headphone mix potentiometers is not connected to the remaining ground plane/ power input. Place a jumper manually!"
- note removed: "Signal Smoothing ==> DNP (not required)"
- moved on the sheet: C301, C304, C311, C315, C318, D302, D303, D304, D305, R303, R304, R309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
