File: schematics/c3lingo_unit-assembly/c3lingo_unit-mix_io/c3lingo_unit-mix_io.kicad_pcb (KiCad board)
At the start: 2 copper layers, 80 x 50 mm, 47 parts, among them J201 Stage Line-In, J202 Mix Line-Out, J203 PowerSupply, J204 Ch1, J205 Ch2, J206 Ch3, SW201 GND Lift, U201 LM833-N, U202 DRV135UA, U203 LM833-N

Commit message: Tidy: Rename hierarchical labels
Connections:
- net /StageSignal renamed /Stage
Changed lines of the file:
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@@
 	(net 2 "+15V")
 	(net 3 "GND")
-	(net 4 "/StageSignal")
+	(net 4 "/Stage")
 	(net 5 "Net-(U201B--)")
 	(net 6 "Net-(C202-Pad2)")
@@
 			(layers "*.Cu" "*.Mask")
 			(remove_unused_layers no)
-			(net 4 "/StageSignal")
+			(net 4 "/Stage")
 			(pinfunction "Pin_3")
 			(pintype "passive")
@@
 			(layers "*.Cu" "*.Mask")
 			(remove_unused_layers no)
-			(net 4 "/StageSignal")
+			(net 4 "/Stage")
 			(pinfunction "Pin_3")
 			(pintype "passive")
@@
 			(layers "*.Cu" "*.Mask")
 			(remove_unused_layers no)
-			(net 4 "/StageSignal")
+			(net 4 "/Stage")
 			(pinfunction "Pin_3")
 			(pintype "passive")
@@
 			(layers "*.Cu" "*.Mask")
 			(remove_unused_layers no)
-			(net 4 "/StageSignal")
+			(net 4 "/Stage")
 			(pinfunction "Pin_3")
 			(pintype "passive")
@@
 			(layers "F.Cu" "F.Paste" "F.Mask")
 			(roundrect_rratio 0.25)
-			(net 4 "/StageSignal")
+			(net 4 "/Stage")
 			(pintype "output")
 		)
@@
 			(layers "*.Cu" "*.Mask")
 			(remove_unused_layers no)
-			(net 4 "/StageSignal")
+			(net 4 "/Stage")
 			(pinfunction "Pin_3")
 			(pintype "passive")
@@
 			(layers "*.Cu" "*.Mask")
 			(remove_unused_layers no)
-			(net 4 "/StageSignal")
+			(net 4 "/Stage")
 			(pinfunction "Pin_3")
 			(pintype "passive")
@@
 			(layers "*.Cu" "*.Mask")
 			(remove_unused_layers no)
-			(net 4 "/StageSignal")
+			(net 4 "/Stage")
 			(pinfunction "1")
 			(pintype "passive")
@@
 			(layers "F.Cu" "F.Paste" "F.Mask")
 			(roundrect_rratio 0.25)
-			(net 4 "/StageSignal")
+			(net 4 "/Stage")
 			(pintype "passive")
 		)
@@
 			(layers "*.Cu" "*.Mask")
 			(remove_unused_layers no)
-			(net 4 "/StageSignal")
+			(net 4 "/Stage")
 			(pinfunction "2")
 			(pintype "passive")

Commit message: Channel Mixer: Rework muting mechanism
Note: Schematic PDF not updated yet
Parts:
- C207, C210: footprint Capacitor_SMD:C_Elec_4x5.4 -> Capacitor_SMD:CP_Elec_4x5.4
Other:
- board text added: "c3lingo Interpreter Unit Mix I/O v0.3.1 2024-08-30"
- board text removed: "c3lingo Interpreter Unit Mix I/O v0.3.1 2024-07-08"
Changed lines of the file:
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@@
 	(title_block
 		(title "c3lingo interpeter unit -- channel strip")
-		(date "2024-07-07")
-		(rev "v0.3")
+		(date "2024-08-30")
+		(rev "v0.3.1")
 		(company "Jannik Beyerstedt (jtbx)")
 		(comment 1 "Prototype 2")
@@
 		)
 	)
-	(footprint "Capacitor_SMD:C_Elec_4x5.4"
+	(footprint "Capacitor_SMD:CP_Elec_4x5.4"
 		(layer "F.Cu")
 		(at 64 70.4375 90)
-		(descr "SMD capacitor, aluminum electrolytic nonpolar, 4.0x5.4mm")
-		(tags "capacitor electrolyic nonpolar")
+		(descr "SMD capacitor, aluminum electrolytic, Panasonic A5 / Nichicon, 4.0x5.4mm")
+		(tags "capacitor electrolytic")
 		(property "Reference" "C210"
 			(at 0 -3.2 90)
@@
 			)
 		)
-		(property "Footprint" "Capacitor_SMD:C_Elec_4x5.4"
+		(property "Footprint" "Capacitor_SMD:CP_Elec_4x5.4"
 			(at 0 0 90)
 			(unlocked yes)
@@
 		)
 		(fp_line
+			(start -2.75 -1.81)
+			(end -2.75 -1.31)
+			(stroke
+				(width 0.12)
+				(type solid)
+			)
+			(layer "F.SilkS")
+		)
+		(fp_line
+			(start -3 -1.56)
+			(end -2.5 -1.56)
+			(stroke
+				(width 0.12)
+				(type solid)
+			)
+			(layer "F.SilkS")
+		)
+		(fp_line
 			(start -2.26 -1.195563)
 			(end -1.195563 -2.26)
@@
 		)
 		(fp_line
-			(start 3.25 -1.05)
-			(end 3.25 1.05)
+			(start 3.35 -1.05)
+			(end 3.35 1.05)
 			(stroke
 				(width 0.05)
@@
 		(fp_line
 			(start 2.4 -1.05)
-			(end 3.25 -1.05)
+			(end 3.35 -1.05)
 			(stroke
 				(width 0.05)
@@
 		(fp_line
 			(start -2.4 -1.05)
-			(end -3.25 -1.05)
+			(end -3.35 -1.05)
 			(stroke
 				(width 0.05)
@@
 		)
 		(fp_line
-			(start -3.25 -1.05)
-			(end -3.25 1.05)
+			(start -3.35 -1.05)
+			(end -3.35 1.05)
 			(stroke
 				(width 0.05)
@@
 		)
 		(fp_line
-			(start 3.25 1.05)
+			(start 3.35 1.05)
 			(end 2.4 1.05)
 			(stroke
@@
 		)
 		(fp_line
-			(start -3.25 1.05)
+			(start -3.35 1.05)
 			(end -2.4 1.05)
 			(stroke
@@
 		)
 		(fp_line
+			(start -1.374773 -1.2)
+			(end -1.374773 -0.8)
+			(stroke
+				(width 0.1)
+				(type solid)
+			)
+			(layer "F.Fab")
+		)
+		(fp_line
 			(start -2.15 -1.15)
 			(end -1.15 -2.15)
@@
 		)
 		(fp_line
+			(start -1.574773 -1)
+			(end -1.174773 -1)
+			(stroke
+				(width 0.1)
+				(type solid)
+			)
+			(layer "F.Fab")
+		)
+		(fp_line
 			(start -2.15 1.15)
 			(end -1.15 2.15)
@@
 		)
 		(pad "1" smd roundrect
-			(at -1.675 0 90)
-			(size 2.65 1.6)
+			(at -1.8 0 90)
+			(size 2.6 1.6)
 			(layers "F.Cu" "F.Paste" "F.Mask")
 			(roundrect_rratio 0.15625)
@@
 		)
 		(pad "2" smd roundrect
-			(at 1.675 0 90)
-			(size 2.65 1.6)
+			(at 1.8 0 90)
+			(size 2.6 1.6)
 			(layers "F.Cu" "F.Paste" "F.Mask")
 			(roundrect_rratio 0.15625)
@@
 			(pintype "passive")
 		)
-		(model "${KICAD8_3DMODEL_DIR}/Capacitor_SMD.3dshapes/C_Elec_4x5.4.wrl"
+		(model "${KICAD8_3DMODEL_DIR}/Capacitor_SMD.3dshapes/CP_Elec_4x5.4.wrl"
 			(offset
 				(xyz 0 0 0)
@@
 		)
 	)
-	(footprint "Capacitor_SMD:C_Elec_4x5.4"
+	(footprint "Capacitor_SMD:CP_Elec_4x5.4"
 		(layer "F.Cu")
 		(at 64 79.5625 -90)
-		(descr "SMD capacitor, aluminum electrolytic nonpolar, 4.0x5.4mm")
-		(tags "capacitor electrolyic nonpolar")
+		(descr "SMD capacitor, aluminum electrolytic, Panasonic A5 / Nichicon, 4.0x5.4mm")
+		(tags "capacitor electrolytic")
 		(property "Reference" "C207"
 			(at 0 -3.2 -90)
@@
 			)
 		)
-		(property "Footprint" "Capacitor_SMD:C_Elec_4x5.4"
+		(property "Footprint" "Capacitor_SMD:CP_Elec_4x5.4"
 			(at 0 0 -90)
 			(unlocked yes)
@@
 		)
 		(fp_line
+			(start -3 -1.56)
+			(end -2.5 -1.56)
+			(stroke
+				(width 0.12)
+				(type solid)
+			)
+			(layer "F.SilkS")
+		)
+		(fp_line
+			(start -2.75 -1.81)
+			(end -2.75 -1.31)
+			(stroke
+				(width 0.12)
+				(type solid)
+			)
+			(layer "F.SilkS")
+		)
+		(fp_line
 			(start -1.195563 -2.26)
 			(end 2.26 -2.26)
@@
 		)
 		(fp_line
-			(start -3.25 1.05)
+			(start -3.35 1.05)
 			(end -2.4 1.05)
 			(stroke
@@
 		)
 		(fp_line
-			(start 3.25 1.05)
+			(start 3.35 1.05)
 			(end 2.4 1.05)
 			(stroke
@@
 		)
 		(fp_line
-			(start -3.25 -1.05)
-			(end -3.25 1.05)
+			(start -3.35 -1.05)
+			(end -3.35 1.05)
 			(stroke
 				(width 0.05)
@@
 		(fp_line
 			(start -2.4 -1.05)
-			(end -3.25 -1.05)
+			(end -3.35 -1.05)
 			(stroke
 				(width 0.05)
@@
 		(fp_line
 			(start 2.4 -1.05)
-			(end 3.25 -1.05)
+			(end 3.35 -1.05)
 			(stroke
 				(width 0.05)
@@
 		)
 		(fp_line
-			(start 3.25 -1.05)
-			(end 3.25 1.05)
+			(start 3.35 -1.05)
+			(end 3.35 1.05)
 			(stroke
 				(width 0.05)
@@
 		)
 		(fp_line
+			(start -1.574773 -1)
+			(end -1.174773 -1)
+			(stroke
+				(width 0.1)
+				(type solid)
+			)
+			(layer "F.Fab")
+		)
+		(fp_line
 			(start -2.15 -1.15)
 			(end -2.15 1.15)
@@
 		)
 		(fp_line
+			(start -1.374773 -1.2)
+			(end -1.374773 -0.8)
+			(stroke
+				(width 0.1)
+				(type solid)
+			)
+			(layer "F.Fab")
+		)
+		(fp_line
 			(start -1.15 -2.15)
 			(end 2.15 -2.15)
@@
 		)
 		(pad "1" smd roundrect
-			(at -1.675 0 270)
-			(size 2.65 1.6)
+			(at -1.8 0 270)
+			(size 2.6 1.6)
 			(layers "F.Cu" "F.Paste" "F.Mask")
 			(roundrect_rratio 0.15625)
@@
 		)
 		(pad "2" smd roundrect
-			(at 1.675 0 270)
-			(size 2.65 1.6)
+			(at 1.8 0 270)
+			(size 2.6 1.6)
 			(layers "F.Cu" "F.Paste" "F.Mask")
 			(roundrect_rratio 0.15625)
@@
 			(pintype "passive")
 		)
-		(model "${KICAD8_3DMODEL_DIR}/Capacitor_SMD.3dshapes/C_Elec_4x5.4.wrl"
+		(model "${KICAD8_3DMODEL_DIR}/Capacitor_SMD.3dshapes/CP_Elec_4x5.4.wrl"
 			(offset
 				(xyz 0 0 0)
@@
 		)
 		(property "Value" "GND Lift"
-			(at 10.12 1.54 360)
+			(at 10.12 1.54 0)
 			(layer "F.SilkS")
 			(effects
@@
 		(layer "Edge.Cuts")
 	)
-	(gr_text "c3lingo Interpreter Unit\nMix I/O\nv0.3.1 2024-07-08"
+	(gr_text "c3lingo Interpreter Unit\nMix I/O\nv0.3.1 2024-08-30"
 		(at 100.5 85.5 0)
 		(layer "B.SilkS")

Commit message: Channel: Change to single channel potentiometers
Other:
- board text added: "c3lingo Interpreter Unit Mix I/O v0.3.2 2024-09-06"
- board text removed: "c3lingo Interpreter Unit Mix I/O v0.3.1 2024-08-30"
Changed lines of the file:
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@@
 	(title_block
 		(title "c3lingo interpeter unit -- channel strip")
-		(date "2024-08-30")
-		(rev "v0.3.1")
+		(date "2024-09-06")
+		(rev "v0.3.2")
 		(company "Jannik Beyerstedt (jtbx)")
 		(comment 1 "Prototype 2")
@@
 		(tags "capacitor handsolder")
 		(property "Reference" "C202"
-			(at 0 -1.43 -90)
+			(at 0 -1.43 90)
 			(layer "F.SilkS")
+			(hide yes)
 			(effects
 				(font
@@
 		)
 		(property "Value" "220pF"
-			(at 0 1.43 -90)
+			(at 0 1.43 90)
 			(layer "F.Fab")
 			(effects
@@
 		)
 		(fp_text user "${REFERENCE}"
-			(at 0 0 -90)
+			(at 0 0 90)
 			(layer "F.Fab")
 			(effects
@@
 			(at 0 -1.43 0)
 			(layer "F.SilkS")
+			(hide yes)
 			(effects
 				(font
@@
 			(at 0 1.8 -90)
 			(layer "B.SilkS")
+			(hide yes)
 			(effects
 				(font
@@
 			(at 0 1.8 -90)
 			(layer "B.SilkS")
+			(hide yes)
 			(effects
 				(font
@@
 		(layer "Edge.Cuts")
 	)
-	(gr_text "c3lingo Interpreter Unit\nMix I/O\nv0.3.1 2024-08-30"
+	(gr_text "c3lingo Interpreter Unit\nMix I/O\nv0.3.2 2024-09-06"
 		(at 100.5 85.5 0)
 		(layer "B.SilkS")

Commit message: Move potentiometers down, fix JLC PCB components
- Fix JLC PCB component orientation
- Add do-not-populate to all THD components
- Fix JLC part selection, tweak values to be standard components
Other:
- board text added: "c3lingo Interpreter Unit Mix I/O v0.3.3 2024-09-08"
- board text removed: "c3lingo Interpreter Unit Mix I/O v0.3.2 2024-09-06"
Changed lines of the file:
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@@
 	(paper "A4" portrait)
 	(title_block
-		(title "c3lingo interpeter unit -- channel strip")
-		(date "2024-09-06")
-		(rev "v0.3.2")
+		(title "c3lingo interpeter unit -- main I/O")
+		(date "2024-09-08")
+		(rev "v0.3.3")
 		(company "Jannik Beyerstedt (jtbx)")
 		(comment 1 "Prototype 2")
@@
 			)
 		)
-		(property "LCSC Part #" "C3001226"
+		(property "LCSC Part #" "C3343"
 			(at 0 0 90)
 			(unlocked yes)
@@
 			)
 		)
+		(property "JLCPCB Rotation Offset" "180"
+			(at 0 0 0)
+			(unlocked yes)
+			(layer "F.Fab")
+			(hide yes)
+			(effects
+				(font
+					(size 1 1)
+					(thickness 0.15)
+				)
+			)
+		)
 		(property ki_fp_filters "CP_*")
 		(sheetname "Root")
@@
 		(sheetname "Root")
 		(sheetfile "c3lingo_unit-mix_io.kicad_sch")
-		(attr through_hole)
+		(attr through_hole dnp)
 		(fp_line
 			(start -1.14 5.96)
@@
 			)
 		)
-		(property "LCSC Part #" "C3001226"
+		(property "LCSC Part #" "C3343"
+			(at 0 0 -90)
+			(unlocked yes)
+			(layer "F.Fab")
+			(hide yes)
+			(effects
+				(font
+					(size 1 1)
+					(thickness 0.15)
+				)
+			)
+		)
+		(property "JLCPCB Rotation Offset" "180"
 			(at 0 0 -90)
 			(unlocked yes)
@@
 		(sheetname "Root")
 		(sheetfile "c3lingo_unit-mix_io.kicad_sch")
-		(attr through_hole)
+		(attr through_hole dnp)
 		(fp_line
 			(start -1.14 4.96)
@@
 		(layer "Edge.Cuts")
 	)
-	(gr_text "c3lingo Interpreter Unit\nMix I/O\nv0.3.2 2024-09-06"
+	(gr_text "c3lingo Interpreter Unit\nMix I/O\nv0.3.3 2024-09-08"
 		(at 100.5 85.5 0)
 		(layer "B.SilkS")
