File: schematics/c3lingo_unit-assembly/c3lingo_unit-channel_io/c3lingo_unit-channel_io.kicad_sch (KiCad schematic)
At the start: 39 parts, among them J601 Mic X In, J602 Headphone X, J603 Interconnect, U601 NE5534, U602 TPA6111A2

Commit message: Refactor: Rename component rotation
The latest release of the (JLC PCB) Fabrication Toolkit plugin needs the rotation offset field to be named "FT Rotation Offset"
Parts:
- C602, C605, C606, C607, C608, C609, C610, C611, C614, D601, D602, D603, D604: FT Rotation Offset (none) -> 180; JLCPCB Rotation Offset 180 -> (none)
Changed lines of the file:
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@@
 			)
 		)
-		(property "JLCPCB Rotation Offset" ""
+		(property "FT Rotation Offset" ""
 			(at 95.25 76.2 0)
 			(effects
@@
 			)
 		)
-		(property "JLCPCB Rotation Offset" ""
+		(property "FT Rotation Offset" ""
 			(at 80.01 63.5 0)
 			(effects
@@
 			)
 		)
-		(property "JLCPCB Rotation Offset" ""
+		(property "FT Rotation Offset" ""
 			(at 106.68 88.9 0)
 			(effects
@@
 			)
 		)
-		(property "JLCPCB Rotation Offset" ""
+		(property "FT Rotation Offset" ""
 			(at 76.2 76.2 0)
 			(effects
@@
 			)
 		)
-		(property "JLCPCB Rotation Offset" ""
+		(property "FT Rotation Offset" ""
 			(at 80.01 88.9 0)
 			(effects
@@
 			)
 		)
-		(property "JLCPCB Rotation Offset" ""
+		(property "FT Rotation Offset" ""
 			(at 106.68 63.5 0)
 			(effects
@@
 			)
 		)
-		(property "JLCPCB Rotation Offset" ""
+		(property "FT Rotation Offset" ""
 			(at 100.33 101.6 90)
 			(effects
@@
 			)
 		)
-		(property "JLCPCB Rotation Offset" ""
+		(property "FT Rotation Offset" ""
 			(at 100.33 43.18 90)
 			(effects
@@
 			)
 		)
-		(property "JLCPCB Rotation Offset" ""
+		(property "FT Rotation Offset" ""
 			(at 224.79 86.36 0)
 			(effects
@@
 			)
 		)
-		(property "JLCPCB Rotation Offset" "180"
+		(property "FT Rotation Offset" "180"
 			(at 232.41 106.68 0)
 			(effects
@@
 			)
 		)
-		(property "JLCPCB Rotation Offset" "180"
+		(property "FT Rotation Offset" "180"
 			(at 248.92 81.28 0)
 			(effects
@@
 			)
 		)
-		(property "JLCPCB Rotation Offset" ""
+		(property "FT Rotation Offset" ""
 			(at 198.12 86.36 90)
 			(effects
@@
 			)
 		)
-		(property "JLCPCB Rotation Offset" "180"
+		(property "FT Rotation Offset" "180"
 			(at 248.92 86.36 0)
 			(effects
@@
 			)
 		)
-		(property "JLCPCB Rotation Offset" ""
+		(property "FT Rotation Offset" ""
 			(at 38.1 69.85 0)
 			(effects
@@
 			)
 		)
-		(property "JLCPCB Rotation Offset" ""
+		(property "FT Rotation Offset" ""
 			(at 38.1 82.55 0)
 			(effects
@@
 			)
 		)
-		(property "JLCPCB Rotation Offset" "180"
+		(property "FT Rotation Offset" "180"
 			(at 55.88 78.74 0)
 			(effects
@@
 			)
 		)
-		(property "JLCPCB Rotation Offset" ""
+		(property "FT Rotation Offset" ""
 			(at 208.28 72.39 0)
 			(effects
@@
 			)
 		)
-		(property "JLCPCB Rotation Offset" ""
+		(property "FT Rotation Offset" ""
 			(at 198.12 81.28 90)
 			(effects
@@
 			)
 		)
-		(property "JLCPCB Rotation Offset" "180"
+		(property "FT Rotation Offset" "180"
 			(at 44.45 63.5 0)
 			(effects
@@
 			)
 		)
-		(property "JLCPCB Rotation Offset" "180"
+		(property "FT Rotation Offset" "180"
 			(at 66.04 57.15 0)
 			(effects
@@
 			)
 		)
-		(property "JLCPCB Rotation Offset" "180"
+		(property "FT Rotation Offset" "180"
 			(at 54.61 57.15 0)
 			(effects
@@
 			)
 		)
-		(property "JLCPCB Rotation Offset" ""
+		(property "FT Rotation Offset" ""
 			(at 232.41 57.15 90)
 			(effects
@@
 			)
 		)
-		(property "JLCPCB Rotation Offset" "180"
+		(property "FT Rotation Offset" "180"
 			(at 189.23 81.28 0)
 			(effects
@@
 			)
 		)
-		(property "JLCPCB Rotation Offset" "180"
+		(property "FT Rotation Offset" "180"
 			(at 44.45 88.9 0)
 			(effects
@@
 			)
 		)
-		(property "JLCPCB Rotation Offset" "180"
+		(property "FT Rotation Offset" "180"
 			(at 240.03 49.53 0)
 			(effects
@@
 			)
 		)
-		(property "JLCPCB Rotation Offset" "180"
+		(property "FT Rotation Offset" "180"
 			(at 66.04 95.25 0)
 			(effects
@@
 			)
 		)
-		(property "JLCPCB Rotation Offset" "180"
+		(property "FT Rotation Offset" "180"
 			(at 54.61 95.25 0)
 			(effects
@@
 			)
 		)
-		(property "JLCPCB Rotation Offset" "180"
+		(property "FT Rotation Offset" "180"
 			(at 189.23 86.36 0)
 			(effects
@@
 			)
 		)
-		(property "JLCPCB Rotation Offset" ""
+		(property "FT Rotation Offset" ""
 			(at 106.68 58.42 90)
 			(effects
@@
 			)
 		)
-		(property "JLCPCB Rotation Offset" ""
+		(property "FT Rotation Offset" ""
 			(at 208.28 95.25 0)
 			(effects

Commit message: Channel I/O: Mark phantom power testpoint as DNP
It's just a footprint to solder a wire on and no component to populate.
Parts:
- TP601: now not fitted
Changed lines of the file:
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@@
 		(in_bom yes)
 		(on_board yes)
-		(dnp no)
+		(dnp yes)
 		(fields_autoplaced yes)
 		(property "Reference" "TP601"

Commit message: Channel I/O: Fix value of C601
Parts:
- C601: value 220p -> 330p; footprint Capacitor_SMD:C_0402_1005Metric_Pad0.74x0.62mm_HandSolder -> Capacitor_SMD:C_0603_1608Metric_Pad1.08x0.95mm_HandSolder; LCSC Part # C107001 -> C1664
Other:
- note added: "Errata to v0.4.0: - C601: Replace with 330p"
Changed lines of the file:
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@@
 	(title_block
 		(title "c3lingo interpeter unit -- channel I/O")
-		(date "2025-08-26")
-		(rev "v0.4.0")
+		(date "2025-08-31")
+		(rev "v0.4.1")
 		(company "Jannik Beyerstedt (jtbx)")
-		(comment 1 "Prototype 3")
+		(comment 1 "Prototype 3 + Errata")
 	)
 	(text "Mic Preamp\nGain: 30 dB\nLP-Filter: 10 kHz"
@@
 		)
 	)
+	(text "Errata to v0.4.0:\n- C601: Replace with 330p"
+		(exclude_from_sim no)
+		(at 177.8 164.084 0)
+		(effects
+			(font
+				(size 1.27 1.27)
+			)
+			(justify left bottom)
+		)
+	)
 	(text "Phantom Power\n(48V)"
 		(exclude_from_sim no)
@@
 			)
 		)
-		(property "Value" "220p"
+		(property "Value" "330p"
 			(at 106.68 54.5408 90)
 			(effects
@@
 			)
 		)
-		(property "Footprint" "Capacitor_SMD:C_0402_1005Metric_Pad0.74x0.62mm_HandSolder"
+		(property "Footprint" "Capacitor_SMD:C_0603_1608Metric_Pad1.08x0.95mm_HandSolder"
 			(at 110.49 57.4548 0)
 			(effects
@@
 			)
 		)
-		(property "LCSC Part #" "C107001"
+		(property "LCSC Part #" "C1664"
 			(at 106.68 58.42 0)
 			(effects

Commit message: Channel-IO: Use horizontal IDC connector
Parts:
- J603: footprint Connector_IDC:IDC-Header_2x04_P2.54mm_Vertical -> Connector_IDC:IDC-Header_2x04_P2.54mm_Horizontal
Changed lines of the file:
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@@
 	(title_block
 		(title "c3lingo interpeter unit -- channel I/O")
-		(date "2025-08-31")
-		(rev "v0.4.1")
+		(date "2025-09-29")
+		(rev "v0.5.0-dev")
 		(company "Jannik Beyerstedt (jtbx)")
-		(comment 1 "Prototype 3 + Errata")
+		(comment 1 "Prototype 3b")
 	)
 	(text "Mic Preamp\nGain: 30 dB\nLP-Filter: 10 kHz"
@@
 			)
 		)
-		(property "Footprint" "Connector_IDC:IDC-Header_2x04_P2.54mm_Vertical"
+		(property "Footprint" "Connector_IDC:IDC-Header_2x04_P2.54mm_Horizontal"
 			(at 63.5 175.26 0)
 			(effects
