File: schematics/c3lingo_unit-assembly/c3lingo_unit-channel_io/c3lingo_unit-channel_io.kicad_sch (KiCad schematic)
At the start: 39 parts, among them J601 Mic X In, J602 Headphone X, J603 Interconnect, U601 NE5534, U602 TPA6111A2

Commit message: Channel: Swap mic and headphone signal on IDC connector
Connections:
- net Headphone: now also J603.8 (Pin_8); no longer J603.6 (Pin_6)
- net MicPre: now also J603.6 (Pin_6); no longer J603.8 (Pin_8)
Changed lines of the file:
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@@
 	(hierarchical_label "MicPre"
 		(shape output)
-		(at 73.66 161.29 90)
+		(at 77.47 161.29 90)
 		(effects
 			(font
@@
 	(hierarchical_label "Headphone"
 		(shape input)
-		(at 77.47 161.29 90)
+		(at 73.66 161.29 90)
 		(effects
 			(font

Commit message: chore: Bump version number, plot schematic
Other:
- company: Jannik Beyerstedt (jtbx) -> c3lingo/ c3voc: jtbx and collaborators
Changed lines of the file:
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@@
 	(title_block
 		(title "c3lingo interpeter unit -- channel I/O")
-		(date "2025-09-29")
-		(rev "v0.5.0-dev")
-		(company "Jannik Beyerstedt (jtbx)")
-		(comment 1 "Prototype 3b")
+		(date "2025-10-16")
+		(rev "v1.0.0")
+		(company "c3lingo/ c3voc: jtbx and collaborators")
 	)
 	(text "Mic Preamp\nGain: 30 dB\nLP-Filter: 10 kHz"
