File: schematics/c3lingo_unit-assembly/c3lingo_unit-assembly.kicad_sch (KiCad schematic)
At the start: 0 parts

Commit message: chore: Bump version number, plot schematic
Other:
- company: Jannik Beyerstedt (jtbx) -> c3lingo/ c3voc: jtbx and collaborators
Changed lines of the file:
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@@
 	(title_block
 		(title "c3lingo interpeter unit")
-		(date "2025-09-08")
-		(rev "v0.4.1")
-		(company "Jannik Beyerstedt (jtbx)")
-		(comment 1 "Prototype 3 + Errata")
+		(date "2025-10-16")
+		(rev "v1.0.0")
+		(company "c3lingo/ c3voc: jtbx and collaborators")
 	)
 	(text "Make the ERC happy"
